Commit message: Correct camera/lidar geometry against the real Seeed kit; rebuild lidar mount from scratch; regenerate both URDFs from the verified USD
Camera variant: fixed a baked 180deg root-rotation mirror bug and
replaced the wrong GoPro-pedestal camera mount with a flush bracket
matching Seeed's real product photo.

Lidar variant: deleted and rebuilt usd/lekiwi_lidar.usd from scratch on
real Slamtec RPLIDAR A1M8 datasheet dimensions -- correct obstruction
avoidance (the real motor-controller board, not a phantom reference),
a real 25mm 3D-printable mount block with M3/M2.5 heat-set-insert
holes matched to the base plate's actual hole grid, and the RPLIDAR
itself modeled as a real paddle shape (circle + boss union) instead of
a box.

Wheel geometry: all three wheels set to an explicit 118mm
closest-approach-to-center target, applied as a precise radial scale
with drivetrain hardware (motor mounts, servos) moved to match.

urdf/lekiwi_cam.urdf and urdf/lekiwi_lidar.urdf regenerated entirely by
extracting geometry, mass/inertia, and joints directly from the
corrected USD files, so the URDF and USD share one source of truth.
Adds the ~110 fresh meshes this requires.

Co-Authored-By: Claude Sonnet 5 <noreply@anthropic.com>

File: urdf/lekiwi_lidar.urdf (robot description, URDF)
Before this commit: robot LeKiwi, 28 links, 27 joints
Links:
- removed link Base_08q_v1
- removed link Battery___Battery_5_2_Ah_DC5521_Plug_v2
- removed link Bottom_V2_v3
- removed link ST3215_Servo_Motor_v1
- removed link ST3215_Servo_Motor_v1_1
- removed link ST3215_Servo_Motor_v1_2
- removed link Top_V2_v2
- removed link WaveShare_Mounting_Plate_01d_v1
- removed link a_4_Omni_Directional_Wheel_Single_Body_v1
- removed link a_4_Omni_Directional_Wheel_Single_Body_v1_1
- removed link a_4_Omni_Directional_Wheel_Single_Body_v1_2
- removed link a_94868A713_NO_THREADS_Female_Threaded_Hex_Standoff
- removed link a_94868A713_NO_THREADS_Female_Threaded_Hex_Standoff_1
- removed link a_94868A713_NO_THREADS_Female_Threaded_Hex_Standoff_2
- removed link a_94868A713_NO_THREADS_Female_Threaded_Hex_Standoff_3
- removed link a_94868A713_NO_THREADS_Female_Threaded_Hex_Standoff_4
- removed link a_94868A713_NO_THREADS_Female_Threaded_Hex_Standoff_5
- removed link base_plate_layer1_v5
- removed link base_plate_layer2_v3
- removed link drive_motor_mount_v11
- removed link drive_motor_mount_v11_1
- removed link drive_motor_mount_v11_2
- removed link lipo_battery_mount_v3
- removed link omni_wheel_mount_v5
- removed link omni_wheel_mount_v5_1
- removed link omni_wheel_mount_v5_2
- removed link rplidar_a1m8_link
- removed link servo_controller_mount_v3
- added link base, mass 7.931429; collision mesh filename=meshes/lidar_base_Battery___Battery_5_2_Ah_DC5521_Plug_v2_1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 scale=0.001 0.001 0.001; collision mesh filename=meshes/lidar_base_Bottom_V2_v3_1.stl scale=0.001 0.001 0.001
- added link lidar_assembly, mass 0.259245; collision mesh filename=meshes/lidar_lidar_assembly_lidar_mount_block_v1_1.stl scale=0.001 0.001 0.001; collision mesh filename=meshes/lidar_lidar_assembly_rplidar_a1m8_base_1.stl scale=0.001 0.001 0.001
- added link wheel_back, mass 1.477856; collision mesh filename=meshes/lidar_wheel_back_a__Omni_Directional_Wheel_Single_Bo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 scale=0.001 0.001 0.001; collision mesh filename=meshes/lidar_wheel_back_omni_wheel_mount_v5_2_1.stl scale=0.001 0.001 0.001
- added link wheel_left, mass 1.477856; collision mesh filename=meshes/lidar_wheel_left_a__Omni_Directional_Wheel_Single_Bo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 scale=0.001 0.001 0.001; collision mesh filename=meshes/lidar_wheel_left_omni_wheel_mount_v5_1.stl scale=0.001 0.001 0.001
- added link wheel_right, mass 1.477856; collision mesh filename=meshes/lidar_wheel_right_a__Omni_Directional_Wheel_Single_B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 scale=0.001 0.001 0.001; collision mesh filename=meshes/lidar_wheel_right_omni_wheel_mount_v5_1_1.stl scale=0.001 0.001 0.001
Joints:
- removed joint Base_08q_v1_Rigid_43
- removed joint Bottom_V2_v3_Rigid_24
- removed joint ST3215_Servo_Motor_v1_1_Revolute_62
- removed joint ST3215_Servo_Motor_v1_2_Revolute_60
- removed joint ST3215_Servo_Motor_v1_Revolute_64
- removed joint a_94868A713_NO_THREADS_Female_Threaded_Hex_Standoff_Rigid_21
- removed joint base_plate_layer1_v5_Rigid_15
- removed joint base_plate_layer1_v5_Rigid_18
- removed joint base_plate_layer1_v5_Rigid_20
- removed joint base_plate_layer1_v5_Rigid_30
- removed joint base_plate_layer1_v5_Rigid_31
- removed joint base_plate_layer1_v5_Rigid_32
- removed joint base_plate_layer1_v5_Rigid_69
- removed joint base_plate_layer1_v5_Rigid_70
- removed joint base_plate_layer1_v5_baseplate2bottom_mount
- removed joint base_plate_layer1_v5_baseplate2left_mount
- removed joint base_plate_layer1_v5_baseplate2right_mount
- removed joint base_plate_layer2_v3_Rigid_22
- removed joint base_plate_layer2_v3_Rigid_42
- removed joint drive_motor_mount_v11_1_Rigid_35
- removed joint drive_motor_mount_v11_2_Rigid_2
- removed joint drive_motor_mount_v11_Rigid_39
- removed joint lipo_battery_mount_v3_Rigid_19
- removed joint omni_wheel_mount_v5_1_Rigid_63
- removed joint omni_wheel_mount_v5_2_Rigid_61
- removed joint omni_wheel_mount_v5_Rigid_65
- removed joint rplidar_a1m8_joint
- added joint fix_lidar_assembly: type fixed, parent base, child lidar_assembly, origin xyz=-0.00038116 0.01483253 0.05700000 rpy=0.00000000 0.00000000 -0.00409005
- added joint fix_wheel_back: type fixed, parent base, child wheel_back, origin xyz=0.00060083 -0.11816273 0.01786001 rpy=-1.57079659 -0.00000006 0.00000020
- added joint fix_wheel_left: type fixed, parent base, child wheel_left, origin xyz=-0.10277865 0.05858054 0.01786001 rpy=-1.57079609 -0.00000010 0.00000013
- added joint fix_wheel_right: type fixed, parent base, child wheel_right, origin xyz=0.10143365 0.05937464 0.01786001 rpy=-1.57079676 -0.00000007 -0.00000014
