Commit message: Correct camera/lidar geometry against the real Seeed kit; rebuild lidar mount from scratch; regenerate both URDFs from the verified USD
Camera variant: fixed a baked 180deg root-rotation mirror bug and
replaced the wrong GoPro-pedestal camera mount with a flush bracket
matching Seeed's real product photo.

Lidar variant: deleted and rebuilt usd/lekiwi_lidar.usd from scratch on
real Slamtec RPLIDAR A1M8 datasheet dimensions -- correct obstruction
avoidance (the real motor-controller board, not a phantom reference),
a real 25mm 3D-printable mount block with M3/M2.5 heat-set-insert
holes matched to the base plate's actual hole grid, and the RPLIDAR
itself modeled as a real paddle shape (circle + boss union) instead of
a box.

Wheel geometry: all three wheels set to an explicit 118mm
closest-approach-to-center target (a user-picked design decision, not
photo-derived), applied as a precise radial scale with drivetrain
hardware (motor mounts, servos) moved to match.

urdf/lekiwi_cam.urdf and urdf/lekiwi_lidar.urdf regenerated entirely by
extracting geometry, mass/inertia, and joints directly from the
corrected USD files, replacing the old independently-traced OnShape
lineage that had drifted out of sync with it.

BoM.md and plan.md updated for the lidar mount hardware and the
domain-randomization spec.

Co-Authored-By: Claude Sonnet 5 <noreply@anthropic.com>

File: urdf/lekiwi_cam.urdf (robot description, URDF)
Before this commit: robot LeKiwi, 29 links, 28 joints
Links:
- removed link Base_08q_v1
- removed link Battery___Battery_5_2_Ah_DC5521_Plug_v2
- removed link Bottom_V2_v3
- removed link Camera_Bracket
- removed link ST3215_Servo_Motor_v1
- removed link ST3215_Servo_Motor_v1_1
- removed link ST3215_Servo_Motor_v1_2
- removed link Top_V2_v2
- removed link WaveShare_Mounting_Plate_01d_v1
- removed link X10_USB_Camera
- removed link a_4_Omni_Directional_Wheel_Single_Body_v1
- removed link a_4_Omni_Directional_Wheel_Single_Body_v1_1
- removed link a_4_Omni_Directional_Wheel_Single_Body_v1_2
- removed link a_94868A713_NO_THREADS_Female_Threaded_Hex_Standoff
- removed link a_94868A713_NO_THREADS_Female_Threaded_Hex_Standoff_1
- removed link a_94868A713_NO_THREADS_Female_Threaded_Hex_Standoff_2
- removed link a_94868A713_NO_THREADS_Female_Threaded_Hex_Standoff_3
- removed link a_94868A713_NO_THREADS_Female_Threaded_Hex_Standoff_4
- removed link a_94868A713_NO_THREADS_Female_Threaded_Hex_Standoff_5
- removed link base_plate_layer1_v5
- removed link base_plate_layer2_v3
- removed link drive_motor_mount_v11
- removed link drive_motor_mount_v11_1
- removed link drive_motor_mount_v11_2
- removed link lipo_battery_mount_v3
- removed link omni_wheel_mount_v5
- removed link omni_wheel_mount_v5_1
- removed link omni_wheel_mount_v5_2
- removed link servo_controller_mount_v3
- added link base, mass 7.931429; collision mesh filename=meshes/camera_base_Battery___Battery_5_2_Ah_DC5521_Plug_v2_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 scale=0.001 0.001 0.001; collision mesh filename=meshes/camera_base_Bottom_V2_v3_1.stl scale=0.001 0.001 0.001
- added link front_camera, mass 0.001
- added link wheel_back, mass 1.477856; collision mesh filename=meshes/camera_wheel_back_a__Omni_Directional_Wheel_Single_B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 scale=0.001 0.001 0.001; collision mesh filename=meshes/camera_wheel_back_omni_wheel_mount_v5_2_1.stl scale=0.001 0.001 0.001
- added link wheel_left, mass 1.477856; collision mesh filename=meshes/camera_wheel_left_a__Omni_Directional_Wheel_Single_B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 scale=0.001 0.001 0.001; collision mesh filename=meshes/camera_wheel_left_omni_wheel_mount_v5_1.stl scale=0.001 0.001 0.001
- added link wheel_right, mass 1.477856; collision mesh filename=meshes/camera_wheel_right_a__Omni_Directional_Wheel_Single_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 scale=0.001 0.001 0.001; collision mesh filename=meshes/camera_wheel_right_omni_wheel_mount_v5_1_1.stl scale=0.001 0.001 0.001
Joints:
- removed joint Base_08q_v1_Rigid_43
- removed joint Bottom_V2_v3_Rigid_24
- removed joint Camera_Bracket_to_X10_USB_Camera
- removed joint ST3215_Servo_Motor_v1_1_Revolute_62
- removed joint ST3215_Servo_Motor_v1_2_Revolute_60
- removed joint ST3215_Servo_Motor_v1_Revolute_64
- removed joint a_94868A713_NO_THREADS_Female_Threaded_Hex_Standoff_Rigid_21
- removed joint base_plate_layer1_v5_Rigid_15
- removed joint base_plate_layer1_v5_Rigid_18
- removed joint base_plate_layer1_v5_Rigid_20
- removed joint base_plate_layer1_v5_Rigid_30
- removed joint base_plate_layer1_v5_Rigid_31
- removed joint base_plate_layer1_v5_Rigid_32
- removed joint base_plate_layer1_v5_Rigid_69
- removed joint base_plate_layer1_v5_Rigid_70
- removed joint base_plate_layer1_v5_baseplate2bottom_mount
- removed joint base_plate_layer1_v5_baseplate2left_mount
- removed joint base_plate_layer1_v5_baseplate2right_mount
- removed joint base_plate_layer1_v5_camera_bracket
- removed joint base_plate_layer2_v3_Rigid_22
- removed joint base_plate_layer2_v3_Rigid_42
- removed joint drive_motor_mount_v11_1_Rigid_35
- removed joint drive_motor_mount_v11_2_Rigid_2
- removed joint drive_motor_mount_v11_Rigid_39
- removed joint lipo_battery_mount_v3_Rigid_19
- removed joint omni_wheel_mount_v5_1_Rigid_63
- removed joint omni_wheel_mount_v5_2_Rigid_61
- removed joint omni_wheel_mount_v5_Rigid_65
- added joint fix_front_camera: type fixed, parent base, child front_camera, origin xyz=0.00000000 0.11500000 0.02500000 rpy=1.74532296 0.00000000 0.00000000
- added joint fix_wheel_back: type fixed, parent base, child wheel_back, origin xyz=0.00060083 -0.11816273 0.01786001 rpy=-1.57079659 -0.00000006 0.00000020
- added joint fix_wheel_left: type fixed, parent base, child wheel_left, origin xyz=-0.10277865 0.05858054 0.01786001 rpy=-1.57079609 -0.00000010 0.00000013
- added joint fix_wheel_right: type fixed, parent base, child wheel_right, origin xyz=0.10143365 0.05937464 0.01786001 rpy=-1.57079676 -0.00000007 -0.00000014

Commit message: Match camera/lidar FOV at 90deg, replace the X10 with an FOV-published Arducam board, and design a real mounting bracket for it
Lidar: horizontal_fov_range narrowed from the full 360deg sweep to a
forward-facing 90deg window, matching the camera. Caught and fixed a real
bug in the process: mdp/_pure_math.py's angular-jitter functions inferred
angular resolution as 360/num_rays, silently correct only by coincidence at
the old full-circle FOV -- would have understated jitter by 4x at 90deg.
Fixed by threading the sensor's real resolution through explicitly instead,
proven with a new regression test (37/37 passing). Hardcoded ray-count
constants in export_policy.py and the on-robot deploy skeleton updated to
match (360 -> 90).

Camera (sim): the USD's baked-in optics widened from ~53.5deg to exactly
90deg horizontal FOV via a direct pxr edit, also fixing a real latent
aspect-ratio bug (the old vertical_aperture never matched the 640x480 render
resolution at all).

Camera (real hardware): the Seeed X10 -- whose real FOV was never published
anywhere, confirmed again this session -- replaced with an Arducam IMX291
board camera (SKU B0200, ~100degree published FOV). Price could not be
tool-verified (every retailer blocks automated fetches or renders price via
JS); flagged honestly in BoM.md rather than guessed at.

New real mounting bracket (urdf/meshes/camera_mount_bracket_v1.stl, same
trimesh+manifold3d methodology as the lidar mount): base flange bolts to
real holes extracted directly from the base plate mesh, riser holds the
Arducam board via its real datasheet-sourced mounting pattern. A real
collision with the existing servo_controller_mount_v3 was found and fixed
during verification (not shipped and found later) -- the flange was
reshaped from a solid rectangle into a frame routing around it, reverified
clear against every other component on the robot via dense surface-point
sampling. Old placeholder camera geometry deleted from the USD and URDF
(not deactivated, per explicit instruction); front_camera repositioned to
the new bracket's actual face.

BoM.md, plan.md, and plan_log.md updated to match, including a new "Camera
Mount Hardware" section and an honest accounting of the now-unconfirmed
camera price.

Co-Authored-By: Claude Sonnet 5 <noreply@anthropic.com>

File: urdf/lekiwi_cam.urdf (robot description, URDF)
Before this commit: robot LeKiwi, 5 links, 4 joints
Links:
- link base: geometry collision mesh filename=meshes/camera_base_Battery___Battery_5_2_Ah_DC5521_Plug_v2_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 scale=0.001 0.001 0.001; collision mesh filename=meshes/camera_base_Bottom_V2_v3_1.stl scale=0.001 0.001 0.001
